Commit message: Gazebo初步_建图前

File: src/gasrobot_description/urdf/gasrobot/gas_robot.urdf.xacro (robot description, xacro)
@@ -9,11 +9,20 @@
 <!-- 执行器 -->
 <xacro:include filename="$(find gasrobot_description)/urdf/gasrobot/wheel/wheel.urdf.xacro"/>
+<!-- 插件 -->
+<xacro:include filename="$(find gasrobot_description)/urdf/gasrobot/plugins/gasrobot_ros2_control.xacro"/>
+<!-- 下位机参数是从车体中心到车轮中心的半尺寸：半轴距 0.103 m、半轮距 0.133 m。 -->
+<xacro:property name="wheelbase_half" value="0.103"/>
+<xacro:property name="track_half" value="0.133"/>
 <xacro:base_xacro xyz="0.30 0.305 0.07"/>
 <xacro:imu_xacro xyz="-0.065 0.02 0.0"/>
 <xacro:laser_xacro xyz="0.12 0.0 0.07"/>
 <xacro:camera_xacro xyz="0.15 0.0 0.05"/>
-<xacro:wheel_xacro wheel_name="LeftFront_wheel" xyz="0.15 0.18 -0.02"/>
-<xacro:wheel_xacro wheel_name="LeftBack_wheel" xyz="-0.15 0.18 -0.02"/>
-<xacro:wheel_xacro wheel_name="RightFront_wheel" xyz="0.15 -0.18 -0.02"/>
-<xacro:wheel_xacro wheel_name="RightBack_wheel" xyz="-0.15 -0.18 -0.02"/>
+<xacro:wheel_xacro wheel_name="LeftFront_wheel" xyz="${wheelbase_half} ${track_half} -0.02"/>
+<xacro:wheel_xacro wheel_name="LeftBack_wheel" xyz="${-wheelbase_half} ${track_half} -0.02"/>
+<xacro:wheel_xacro wheel_name="RightFront_wheel" xyz="${wheelbase_half} ${-track_half} -0.02"/>
+<xacro:wheel_xacro wheel_name="RightBack_wheel" xyz="${-wheelbase_half} ${-track_half} -0.02"/>
+<xacro:gasrobot_ros2_control/>
+<!-- 接入二维雷达、IMU 与普通 RGB 相机仿真。 -->
+<xacro:include filename="$(find gasrobot_description)/urdf/gasrobot/plugins/gazebo_sensor_plugin.xacro"/>
+<xacro:gazebo_sensor_plugin/>
 </robot>

File: src/gasrobot_description/urdf/gasrobot/mass_inertia.xacro (robot description, xacro)
@@ -1,20 +1,85 @@
 <?xml version="1.0"?>
-<robot xmlns:xacro="http://ros.org/wiki/xacro">
+<robot xmlns:xacro="http://www.ros.org/wiki/xacro">
+    <!-- =========================================================
+         长方体惯量
+         m：质量 kg
+         w：X方向尺寸
+         h：Y方向尺寸
+         d：Z方向尺寸
+         ========================================================= -->
     <xacro:macro name="box_inertia" params="m w h d">
         <inertial>
-            <mass value="${m}" />
-            <inertia ixx="${(m/12) * (h*h + d*d)}" ixy="0.0" ixz="0.0" iyy="${(m/12) * (w*w + d*d)}" iyz="0.0" izz="${(m/12) * (w*w + h*h)}" />
+            <mass value="${m}"/>
+            <inertia
+                ixx="${(m/12.0) * (h*h + d*d)}"
+                ixy="0.0"
+                ixz="0.0"
+                iyy="${(m/12.0) * (w*w + d*d)}"
+                iyz="0.0"
+                izz="${(m/12.0) * (w*w + h*h)}"
+            />
         </inertial>
     </xacro:macro>
+    <!-- =========================================================
+         圆柱体惯量：圆柱轴沿 Z 轴
+         适用于：
+         - 竖直圆柱
+         - 雷达支撑杆
+         - 默认 URDF cylinder
+         m：质量
+         r：半径
+         h：圆柱长度
+         ========================================================= -->
     <xacro:macro name="cylinder_inertia" params="m r h">
         <inertial>
-            <mass value="${m}" />
-            <inertia ixx="${(m/12) * (3*r*r + h*h)}" ixy="0" ixz="0" iyy="${(m/12) * (3*r*r + h*h)}" iyz="0" izz="${(m/2) * (r*r)}" />
+            <mass value="${m}"/>
+            <inertia
+                ixx="${(m/12.0) * (3*r*r + h*h)}"
+                ixy="0.0"
+                ixz="0.0"
+                iyy="${(m/12.0) * (3*r*r + h*h)}"
+                iyz="0.0"
+                izz="${(m/2.0) * r*r}"
+            />
         </inertial>
     </xacro:macro>
+    <!-- =========================================================
+         圆柱体惯量：圆柱轴沿 Y 轴
+         专门适用于车辆轮子。
+         因为轮子旋转轴为 Y：
+             Iyy = 1/2 * m * r²
+         X、Z 为径向：
+             Ixx = Izz
+                 = 1/12 * m * (3r² + h²)
+         ========================================================= -->
+    <xacro:macro name="cylinder_inertia_y" params="m r h">
+        <inertial>
+            <mass value="${m}"/>
+            <inertia
+                ixx="${(m/12.0) * (3*r*r + h*h)}"
+                ixy="0.0"
+                ixz="0.0"
+                iyy="${(m/2.0) * r*r}"
+                iyz="0.0"
+                izz="${(m/12.0) * (3*r*r + h*h)}"
+            />
+        </inertial>
+    </xacro:macro>
+    <!-- =========================================================
+         实心球体惯量
+         三个方向完全相同：
+             I = 2/5 * m * r²
+         ========================================================= -->
     <xacro:macro name="sphere_inertia" params="m r">
         <inertial>
-            <mass value="${m}" />
-            <inertia ixx="${(2/5) * m * (r*r)}" ixy="0.0" ixz="0.0" iyy="${(2/5) * m * (r*r)}" iyz="0.0" izz="${(2/5) * m * (r*r)}" />
+            <mass value="${m}"/>
+            <inertia
+                ixx="${(2.0/5.0) * m * r*r}"
+                ixy="0.0"
+                ixz="0.0"
+                iyy="${(2.0/5.0) * m * r*r}"
+                iyz="0.0"
+                izz="${(2.0/5.0) * m * r*r}"
+            />
         </inertial>
     </xacro:macro>

File: src/gasrobot_description/urdf/gasrobot/sensor/camera.urdf.xacro (robot description, xacro)
@@ -35,4 +35,11 @@
             <xacro:box_inertia m="0.03" w="0.03" h="0.03" d="0.03"/>
         </link>
+        <link name="camera_optical_link"></link>
+        <!-- 机器人的关节,用于组合部件 -->
+        <joint name="camera_optical_link" type="fixed">
+            <parent link="camera_link"/>
+            <child link="camera_optical_link"/>
+            <origin xyz="0 0 0" rpy="${-pi/2} 0.0 ${-pi/2}"/>
+        </joint>
         <!-- 机器人的关节,用于组合部件 -->
         <joint name="camera_joint" type="fixed">

File: src/gasrobot_description/urdf/gasrobot/sensor/laser.urdf.xacro (robot description, xacro)
@@ -72,4 +72,10 @@
             <origin xyz="${xyz}" rpy="0.0 0.0 0.0"/>
         </joint>
+        <gazebo reference="laserSupport_link">
+            <material>Gazebo/Black</material>
+        </gazebo>
+        <gazebo reference="laser_link">
+            <material>Gazebo/Black</material>
+        </gazebo>
     </xacro:macro>
 </robot>

File: src/gasrobot_description/urdf/gasrobot/wheel/wheel.urdf.xacro (robot description, xacro)
@@ -41,4 +41,21 @@
             <axis xyz="0.0 1.0 0.0"/>        <!-- 让轮子绕y轴转动 -->
         </joint>
+        <!-- ==================== Gazebo 参数 ==================== -->
+        <gazebo reference="${wheel_name}_link">
+            <!-- Gazebo 中轮子显示为黑色 -->
+            <material>Gazebo/Black</material>
+            <!--
+                四轮差速底盘转弯时，前后轮存在不可避免的横向滑移。
+                fdir1 指定车轮滚动方向为车体 x 轴：该方向保留较大的驱动摩擦力；
+                与其垂直的横向使用较小摩擦系数，使底盘能够原地转向。
+                如果两个方向都设为 20，四个轮子会横向锁死，只能前后行驶。
+            -->
+            <fdir1>1.0 0.0 0.0</fdir1>
+            <mu1>2.0</mu1>
+            <mu2>0.05</mu2>
+            <!-- 接触刚度与阻尼 -->
+            <kp>10000000000.0</kp>
+            <kd>1.0</kd>
+        </gazebo>
     </xacro:macro>
 </robot>

Commit message: 添加仿真

File: src/gasrobot_description/urdf/gasrobot/gas_robot.urdf.xacro (robot description, xacro)
@@ -1,4 +1,7 @@
 <?xml version="1.0"?>
 <robot xmlns:xacro= "http://www.ros.org/wiki/xacro" name="gas_robot">
+<!-- 实车默认只加载模型；仿真入口显式开启插件并传入控制器配置。 -->
+<xacro:arg name="simulation" default="false"/>
+<xacro:arg name="controllers_file" default=""/>
 <!-- 底盘 -->
 <xacro:include filename="$(find gasrobot_description)/urdf/gasrobot/base.urdf.xacro"/>
@@ -22,7 +25,9 @@
 <xacro:wheel_xacro wheel_name="RightFront_wheel" xyz="${wheelbase_half} ${-track_half} -0.02"/>
 <xacro:wheel_xacro wheel_name="RightBack_wheel" xyz="${-wheelbase_half} ${-track_half} -0.02"/>
-<xacro:gasrobot_ros2_control/>
+<xacro:if value="$(arg simulation)">
+<xacro:gasrobot_ros2_control controllers_file="$(arg controllers_file)"/>
 <!-- 接入二维雷达、IMU 与普通 RGB 相机仿真。 -->
 <xacro:include filename="$(find gasrobot_description)/urdf/gasrobot/plugins/gazebo_sensor_plugin.xacro"/>
 <xacro:gazebo_sensor_plugin/>
+</xacro:if>
 </robot>

File: src/gasrobot_description/urdf/gasrobot/plugins/gasrobot_ros2_control.xacro (robot description, xacro)
@@ -13,5 +13,5 @@
         </joint>
     </xacro:macro>
-    <xacro:macro name="gasrobot_ros2_control">
+    <xacro:macro name="gasrobot_ros2_control" params="controllers_file">
         <ros2_control name="GasRobotGazeboSystem" type="system">
             <hardware><plugin>gazebo_ros2_control/GazeboSystem</plugin></hardware>
@@ -27,5 +27,5 @@
                 <robot_param>robot_description</robot_param>
                 <robot_param_node>robot_state_publisher</robot_param_node>
-                <parameters>$(find gasrobot_description)/config/gasrobot_ros2_controller.yaml</parameters>
+                <parameters>${controllers_file}</parameters>
                 <ros>
                     <namespace>/</namespace>
